File: KiCad/mata/diodes.kicad_sch (KiCad schematic)
At the start: 98 parts, among them IC1 MCP602-E_P, IC2 MCP602-E_P, IC3 MCP602-E_P, IC4 MCP602-E_P, IC5 MCP602-E_P, IC6 MCP602-E_P, IC7 MCP602-E_P, IC8 MCP602-E_P, J8 Conn_01x08_Pin, J9 Conn_01x08_Pin

Commit message: Hardware: Release rev1.1
Connections:
- net Col1: no longer Dc11.2 (A)
- net Col2: no longer Dc21.2 (A)
- net Col3: no longer Dc31.2 (A)
- net Col4: no longer Dc41.2 (A)
- net Col5: no longer Dc51.2 (A)
- net Col6: no longer Dc61.2 (A)
- net Col7: no longer Dc71.2 (A)
- net Col8: no longer Dc81.2 (A)
- net Row1: no longer Dr11.2 (A)
- net Row2: no longer Dr21.2 (A)
- net Row3: no longer Dr31.2 (A)
- net Row4: no longer Dr41.2 (A)
- net Row5: no longer Dr51.2 (A)
- net Row6: no longer Dr61.2 (A)
- net Row7: no longer Dr71.2 (A)
- net Row8: no longer Dr81.2 (A)
- net DC1: now reaches IC1.1 (VOUTA), Rc1.2, Rx1.1
- net DC1: now also Dc11.2 (A)
- net DC4: now reaches IC1.7 (VOUTB), Rc4.2, Rx4.2
- net DC4: now also Dc41.2 (A)
- net DR1: now reaches IC7.1 (VOUTA), Rr1.2, Rx9.1
- net DR1: now also Dr11.2 (A)
- net DR2: now reaches IC7.7 (VOUTB), Rr2.2, Rx10.2
- net DR2: now also Dr21.2 (A)
- net DC6: now reaches IC4.1 (VOUTA), Rc6.2, Rx6.1
- net DC6: now also Dc61.2 (A)
- net DC7: now reaches IC4.7 (VOUTB), Rc7.2, Rx7.2
- net DC7: now also Dc71.2 (A)
- net DR3: now reaches IC8.1 (VOUTA), Rr3.2, Rx11.1
- net DR3: now also Dr31.2 (A)
- net DC3: now reaches IC3.7 (VOUTB), Rc3.2, Rx3.2
- net DC3: now also Dc31.2 (A)
- net DC5: now reaches IC2.1 (VOUTA), Rc5.2, Rx5.1
- net DC5: now also Dc51.2 (A)
- net DC8: now reaches IC2.7 (VOUTB), Rc8.2, Rx8.2
- net DC8: now also Dc81.2 (A)
- net DR4: now reaches IC8.7 (VOUTB), Rr4.2, Rx12.2
- net DR4: now also Dr41.2 (A)
- net DR8: now reaches IC5.1 (VOUTA), Rr8.2, Rx16.1
- net DR8: now also Dr81.2 (A)
- net DR7: now reaches IC5.7 (VOUTB), Rr7.2, Rx15.2
- net DR7: now also Dr71.2 (A)
- net DC2: now reaches IC3.1 (VOUTA), Rc2.2, Rx2.1
- net DC2: now also Dc21.2 (A)
- net DR6: now reaches IC6.1 (VOUTA), Rr6.2, Rx14.1
- net DR6: now also Dr61.2 (A)
- net DR5: now reaches IC6.7 (VOUTB), Rr5.2, Rx13.2
- net DR5: now also Dr51.2 (A)
Other:
- note added: "Rev 1.1. Poprawienie, z którego napięcia zasilane są diody."
- moved on the sheet: Dc11, Dc21, Dc31, Dc41, Dc51, Dc61, Dc71, Dc81, Dr11, Dr21, Dr31, Dr41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
