File: KiCad/mata/mata.kicad_pcb (KiCad board)
At the start: 2 copper layers, 100 x 100 mm, 159 parts, among them IC1 MCP602-E_P, IC10 IC-WKNSOP8, IC11 IC-WKNSOP8, IC12 LDL1117S33R, IC13 TC1262-3.0VDB, IC2 MCP602-E_P, IC3 MCP602-E_P, IC4 MCP602-E_P, IC5 MCP602-E_P, IC6 MCP602-E_P, IC7 MCP602-E_P, IC8 MCP602-E_P, IC9 ESDALCL6-2SC6, J1 USB_B_Micro, J10 Conn_01x02_Pin, J11 Conn_01x02_Pin, J2 USB_C_Receptacle_PowerOnly_6P, J3 Conn_01x04_Pin, J4 Conn_01x02_Pin, J5 Conn_01x02_Pin, J6 Conn_01x02_Pin, J7 Conn_01x02_Pin, J8 Conn_01x08_Pin, J9 Conn_01x08_Pin, SW1 SW_SPST, SW2 SW_SPST, U1 STM32F303R8Tx, U2 CH340C, Y1 8MHz_CFPS-73_50ppm_-40+85C_3.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

Commit message: Hardware: Release rev1.1
Parts:
- IC12: value LDL1117S33R -> LD1117AS33TR
- R10, R11, R12, R13, R14, R15, R16, R17, R18, R19, R20, R21, R22, R23, R24, R25: value 1k -> 330
- R4: value 5k -> 1k
- Rx1, Rx10, Rx11, Rx12, Rx13, Rx15, Rx16, Rx2, Rx3, Rx4, Rx5, Rx6, Rx7, Rx8, Rx9: value 5k -> 10k
- moved Rr6 0.10 mm to (119.0, 60.9), turned to 90 degrees
- moved Rr7 0.09 mm to (106.9, 60.9), turned to 90 degrees
- turned Rr5 to 90 degrees
Connections:
- Dc11 pad 2: Col1 -> DC1
- Dc21 pad 2: Col2 -> DC2
- Dc31 pad 2: Col3 -> DC3
- Dc41 pad 2: Col4 -> DC4
- Dc51 pad 2: Col5 -> DC5
- Dc61 pad 2: Col6 -> DC6
- Dc71 pad 2: Col7 -> DC7
- Dc81 pad 2: Col8 -> DC8
- Dr11 pad 2: Row1 -> DR1
- Dr21 pad 2: Row2 -> DR2
- Dr31 pad 2: Row3 -> DR3
- Dr41 pad 2: Row4 -> DR4
- Dr51 pad 2: Row5 -> DR5
- Dr61 pad 2: Row6 -> DR6
- Dr71 pad 2: Row7 -> DR7
- Dr81 pad 2: Row8 -> DR8
- IC1 pad 1: Net-(IC1-VOUTA) -> DC1
- IC1 pad 7: Net-(IC1-VOUTB) -> DC4
- IC2 pad 1: Net-(IC2-VOUTA) -> DC5
- IC2 pad 7: Net-(IC2-VOUTB) -> DC8
- IC3 pad 1: Net-(IC3-VOUTA) -> DC2
- IC3 pad 7: Net-(IC3-VOUTB) -> DC3
- IC4 pad 1: Net-(IC4-VOUTA) -> DC6
- IC4 pad 7: Net-(IC4-VOUTB) -> DC7
- IC5 pad 1: Net-(IC5-VOUTA) -> DR8
- IC5 pad 7: Net-(IC5-VOUTB) -> DR7
- IC6 pad 1: Net-(IC6-VOUTA) -> DR6
- IC6 pad 7: Net-(IC6-VOUTB) -> DR5
- IC7 pad 1: Net-(IC7-VOUTA) -> DR1
- IC7 pad 7: Net-(IC7-VOUTB) -> DR2
- IC8 pad 1: Net-(IC8-VOUTA) -> DR3
- IC8 pad 7: Net-(IC8-VOUTB) -> DR4
- Rc1 pad 2: Net-(IC1-VOUTA) -> DC1
- Rc2 pad 2: Net-(IC3-VOUTA) -> DC2
- Rc3 pad 2: Net-(IC3-VOUTB) -> DC3
- Rc4 pad 2: Net-(IC1-VOUTB) -> DC4
- Rc5 pad 2: Net-(IC2-VOUTA) -> DC5
- Rc6 pad 2: Net-(IC4-VOUTA) -> DC6
- Rc7 pad 2: Net-(IC4-VOUTB) -> DC7
- Rc8 pad 2: Net-(IC2-VOUTB) -> DC8
- Rr1 pad 2: Net-(IC7-VOUTA) -> DR1
- Rr2 pad 2: Net-(IC7-VOUTB) -> DR2
- Rr3 pad 2: Net-(IC8-VOUTA) -> DR3
- Rr4 pad 2: Net-(IC8-VOUTB) -> DR4
- Rr5 pad 2: Net-(IC6-VOUTB) -> DR5
- Rr6 pad 2: Net-(IC6-VOUTA) -> DR6
- Rr7 pad 2: Net-(IC5-VOUTB) -> DR7
- Rr8 pad 2: Net-(IC5-VOUTA) -> DR8
- Rx1 pad 1: Net-(IC1-VOUTA) -> DC1
- Rx10 pad 2: Net-(IC7-VOUTB) -> DR2
- Rx11 pad 1: Net-(IC8-VOUTA) -> DR3
- Rx12 pad 2: Net-(IC8-VOUTB) -> DR4
- Rx13 pad 2: Net-(IC6-VOUTB) -> DR5
- Rx14 pad 1: Net-(IC6-VOUTA) -> DR6
- Rx15 pad 2: Net-(IC5-VOUTB) -> DR7
- Rx16 pad 1: Net-(IC5-VOUTA) -> DR8
- Rx2 pad 1: Net-(IC3-VOUTA) -> DC2
- Rx3 pad 2: Net-(IC3-VOUTB) -> DC3
- Rx4 pad 2: Net-(IC1-VOUTB) -> DC4
- Rx5 pad 1: Net-(IC2-VOUTA) -> DC5
- Rx6 pad 1: Net-(IC4-VOUTA) -> DC6
- Rx7 pad 2: Net-(IC4-VOUTB) -> DC7
- Rx8 pad 2: Net-(IC2-VOUTB) -> DC8
- Rx9 pad 1: Net-(IC7-VOUTA) -> DR1
Routing:
- net GND: track 32.8 -> 49.5 mm, vias 52 -> 54
- net DR6: track 0.00 -> 15.2 mm
- net DR4: track 0.00 -> 15.1 mm
- net DR5: track 0.00 -> 14.4 mm
- net DR2: track 0.00 -> 14.4 mm
- net DC4: track 0.00 -> 14.4 mm
- net DC3: track 0.00 -> 14.3 mm
- net DC8: track 0.00 -> 14.3 mm
- net DR7: track 0.00 -> 14.1 mm
- net DC7: track 0.00 -> 14.1 mm
- net DC5: track 0.00 -> 13.3 mm
- net DC6: track 0.00 -> 13.3 mm
- net DC1: track 0.00 -> 13.1 mm
- net DC2: track 0.00 -> 13.1 mm
- net DR1: track 0.00 -> 13.0 mm
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